File: hardware/4.) final version 2003-2015/4.2) version 2006-2011/KiCad/original/AccuSound100_2006-2011_orig_1layer_THT.kicad_pcb (KiCad board)
At the start: 2 copper layers, 200 x 103 mm, 161 parts, among them J1 IN, J2 IN GND, J3 AC~, J4 LED+, J5 LED-, K1 24V SPST 16A, K2 24V SPST 16A, Q1 2SA970, Q10 BF470, Q11 2SA970, Q12 IRF9620, Q13 IRF620, Q14 2SC2240, Q15 BC556B, Q15.1 IRFP240, Q15.2 IRFP240, Q15.3 IRFP240, Q15.4 IRFP240, Q15.5 IRFP240, Q16 BC546B, Q16.1 IRFP9240, Q16.2 IRFP9240, Q16.3 IRFP9240, Q16.4 IRFP9240, Q16.5 IRFP9240, Q17 BC556B, Q18 BF470, Q19 BD129, Q2 2SC2240, Q3 2SA970, Q4 2SC2240, Q5 2SA970, Q6 2SC2240, Q7 2SC2240, Q8 2SA970, Q9 BF469

Commit message: Add files via upload
Parts:
- removed the REF** at (50.0, 158.2)
Other:
- board text added: "Clearance of the high-voltage* zones & tracks to other potentials is 0.8mm except to the edges there is 0,5mm (all other zones & tracks have normal 0,5mm clearance) *(e.g. +UB / -UB / etc.)"
- board text removed: "Freiraum der Hochvolt Flächen zu anderen Potentialen ist 0,8mm außer zu den Rändern da ist 0,5mm (alle anderen Flächen haben normal 0,5mm Freiraum) Abstand der Hochvolt Flächen zueinander (also +UB zu -UB) ist min. 1,5mm"
Changed lines of the file:
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@@
     )
   )
-  (footprint "MountingHole:MountingHole_3.2mm_M3" (layer "F.Cu")
-    (at 50 158.25)
-    (descr "Mounting Hole 3.2mm, no annular, M3")
-    (tags "mounting hole 3.2mm no annular m3")
-    (attr board_only exclude_from_pos_files exclude_from_bom)
-    (fp_text reference "REF**" (at 0 -4.2) (layer "F.SilkS") hide
-      (effects (font (size 1 1) (thickness 0.15)))
-    )
-    (fp_text value "MountingHole_3.2mm_M3" (at 0 4.2) (layer "F.Fab")
-      (effects (font (size 1 1) (thickness 0.15)))
-    )
-    (fp_text user "${REFERENCE}" (at 0.3 0) (layer "F.Fab")
-      (effects (font (size 1 1) (thickness 0.15)))
-    )
-    (fp_circle (center 0 0) (end 3.2 0) (layer "Cmts.User") (width 0.15) (fill none))
-    (fp_circle (center 0 0) (end 3.45 0) (layer "F.CrtYd") (width 0.05) (fill none))
-    (pad "" np_thru_hole circle locked (at 0 0) (size 3.2 3.2) (drill 3.2) (layers *.Cu *.Mask))
-  )
   (footprint "analoghifi:C_Axial_L27mm_D9mm_P27.5mm_Horizontal" (layer "F.Cu")
     (at 223.8 131.8 90)
@@
   (gr_line (start 242 143) (end 42 143) (layer "Edge.Cuts") (width 0.05))
   (gr_line (start 42 143) (end 42 40) (layer "Edge.Cuts") (width 0.05))
-  (gr_text "Freiraum der Hochvolt Flächen zu anderen Potentialen ist 0,8mm \naußer zu den Rändern da ist 0,5mm\n(alle anderen Flächen haben normal 0,5mm Freiraum)\nAbstand der Hochvolt Flächen zueinander (also +UB zu -UB) ist min. 1,5mm" (at 63.5 170.942) (layer "User.1")
-    (effects (font (size 1.5 1.5) (thickness 0.3)))
+  (gr_text "Clearance of the high-voltage* zones & tracks to other potentials is 0.8mm \nexcept to the edges there is 0,5mm\n(all other zones & tracks have normal 0,5mm clearance)\n*(e.g. +UB / -UB / etc.)\n" (at 42.5 166.25) (layer "User.1")
+    (effects (font (size 1.5 1.5) (thickness 0.15)) (justify left))
   )
   (segment (start 223.81 104.31) (end 223.8 104.3) (width 1) (layer "B.Cu") (net 1))

Commit message: Add files via upload
Parts:
- added JP8: Jumper_2_Bridged, analoghifi:R_Axial_very_long_L6.3mm_D2.5mm_P12.7mm_Horizontal_minSilk, F.Cu at (99.0, 97.5)
- C18, C19: footprint analoghifi:CP_Radial_D26.0mm_P10.00mm_SnapIn -> analoghifi:CP_Radial_D26.0mm_P10.00mm_SnapIn_min_Silk
- C2, C3, C9: footprint analoghifi:C_Rect_Mica_L11mm_W3.3mm_P5.90mm -> analoghifi:C_Rect_Mica_Multi_L11.0mm_W3.5mm_P3.50_P5.00_P5.90_P7.50mm
- D17, D18: footprint analoghifi:Diode_long_L6.3mm_D2.5mm_P12.7mm_Horizontal_minSilk -> analoghifi:Diode_long_L6.3mm_D2.5mm_P11,43mm_Horizontal_minSilk
- D22: footprint analoghifi:Diode_L6.3mm_D2.5mm_P10.16mm_Horizontal_minSilk -> analoghifi:D_DO-41_SOD81_very_short_P7.62mm_Horiz_minSilk
- JP5: footprint analoghifi:R_Axial_very_long_L6.3mm_D2.5mm_P12.7mm_Horizontal_minSilk -> analoghifi:R_Axial_even_longer_L6.3mm_D2.5mm_P13.2mm_Horizontal_minSilk
- JP6: footprint analoghifi:R_Axial_very_long_L6.3mm_D2.5mm_P12.7mm_Horizontal_minSilk -> analoghifi:bridge_Wire-1.5mm_diameter
- R24: footprint analoghifi:R_Axial_very_long_L6.3mm_D2.5mm_P12.7mm_Horizontal_minSilk -> analoghifi:R_Axial_DIN0207_L6.3mm_D2.5mm_P10.16mm_Horizontal_minSilk
- R27: footprint analoghifi:R_Axial_very_long_L6.3mm_D2.5mm_P12.7mm_Horizontal_minSilk -> analoghifi:R_Axial_Short_L6.3mm_D2.5mm_P9.0mm_Horiz_minSilk
- moved D22 12.7 mm to (89.1, 96.5)
- moved JP6 4.30 mm to (120.3, 81.0)
- moved C16 1.95 mm to (93.0, 96.0)
- moved J1 1.25 mm to (164.0, 137.0)
- moved J2 1.25 mm to (157.5, 137.0)
- moved C10 1.24 mm to (158.3, 101.2)
- moved C2 1.17 mm to (169.5, 131.5)
- moved D17 1.17 mm to (238.8, 118.5)
- moved D18 1.17 mm to (238.8, 121.7)
- moved C3 1.12 mm to (151.0, 136.5)
- moved Q10 1.00 mm to (185.5, 113.0)
- moved Q9 1.00 mm to (195.0, 113.0)
- moved NTC1 0.80 mm to (148.4, 80.7)
- moved C14 0.76 mm to (227.2, 140.0)
- moved C9 0.75 mm to (143.1, 108.7)
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Connections:
- net Net-(D22-Pad2) renamed /rel_foot
- net Net-(J5-Pad1) renamed /q19_coll
- net Net-(K1-PadA2) renamed /rel_mid
- net Net-(Q19-Pad1) renamed /q19_emit
- K1 pad A1: +UB1 -> /+UB1_1
Routing:
- net GND2: track 37.7 -> 0.00 mm
- net Net-(C23-Pad2): track 55.3 -> 49.8 mm
- net +UB1: track 59.8 -> 54.5 mm
- net Net-(D6-Pad1): track 43.4 -> 38.9 mm
- net /+UB1_1: track 0.00 -> 4.00 mm
- net /driver_pos1: track 46.5 -> 42.9 mm
- net Net-(C9-Pad1): track 3.49 -> 6.02 mm
- net Net-(C16-Pad1): track 11.9 -> 13.8 mm
- net Net-(C3-Pad2): track 20.5 -> 22.3 mm
- net Net-(C1-Pad1): track 21.7 -> 23.5 mm
- net Net-(Q12-Pad1): track 4.84 -> 3.01 mm
- net /+UBv1: track 20.4 -> 19.2 mm
- net AMP Out: track 37.9 -> 36.9 mm
- net /+UBv: track 84.2 -> 83.1 mm
- net Net-(Q10-Pad1): track 2.75 -> 3.75 mm
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Other:
- board text added: "+"
- board text added: "+UB1"
- board text added: "+UB2"
- board text added: "-"
- board text added: "-UB1"
- board text added: "-UB2"
- board text added: "1 2 3"
- board text added: "GND"
- board text added: "IN"
- board text added: "LED"
- board text added: "~"
