File: hardware/4.) final version 2003-2015/4.2) version 2006-2011/KiCad/original/AccuSound100_2006-2011_orig_1layer_THT.kicad_sch (KiCad schematic)
At the start: 158 parts, among them J1 IN, J2 IN GND, J3 AC~, J4 LED+, J5 LED-, K1 24V SPST 16A, K2 24V SPST 16A, Q1 2SA970, Q10 BF470, Q11 2SA970, Q12 IRF9620, Q13 IRF620, Q14 2SC2240, Q15 BC556B, Q15.1 IRFP240, Q15.2 IRFP240, Q15.3 IRFP240, Q15.4 IRFP240, Q15.5 IRFP240, Q16 BC546B, Q16.1 IRFP9240, Q16.2 IRFP9240, Q16.3 IRFP9240, Q16.4 IRFP9240, Q16.5 IRFP9240, Q17 BC556B, Q18 BF470, Q19 BD129, Q2 2SC2240, Q3 2SA970, Q4 2SC2240, Q5 2SA970, Q6 2SC2240, Q7 2SC2240, Q8 2SA970, Q9 BF469

Commit message: Add files via upload
Parts:
- added JP8: Jumper_2_Bridged, analoghifi:R_Axial_very_long_L6.3mm_D2.5mm_P12.7mm_Horizontal_minSilk, symbol analoghifi:Jumper_2_Bridged
- C2, C3, C9: footprint analoghifi:C_Rect_Mica_L11mm_W3.3mm_P5.90mm -> analoghifi:C_Rect_Mica_Multi_L11.0mm_W3.5mm_P3.50_P5.00_P5.90_P7.50mm
- D22: footprint analoghifi:Diode_L6.3mm_D2.5mm_P10.16mm_Horizontal_minSilk -> analoghifi:D_DO-41_SOD81_very_short_P7.62mm_Horiz_minSilk
- JP5: footprint analoghifi:R_Axial_very_long_L6.3mm_D2.5mm_P12.7mm_Horizontal_minSilk -> analoghifi:R_Axial_even_longer_L6.3mm_D2.5mm_P13.2mm_Horizontal_minSilk
- JP6: footprint analoghifi:R_Axial_very_long_L6.3mm_D2.5mm_P12.7mm_Horizontal_minSilk -> analoghifi:bridge_Wire-1.5mm_diameter
- R24: footprint analoghifi:R_Axial_very_long_L6.3mm_D2.5mm_P12.7mm_Horizontal_minSilk -> analoghifi:R_Axial_DIN0207_L6.3mm_D2.5mm_P10.16mm_Horizontal_minSilk
- R27: footprint analoghifi:R_Axial_very_long_L6.3mm_D2.5mm_P12.7mm_Horizontal_minSilk -> analoghifi:R_Axial_Short_L6.3mm_D2.5mm_P9.0mm_Horiz_minSilk
Connections:
- net +UB1: now also JP8.1 (A); no longer K1.A1
- net q19_emit: now reaches Q19.1 (E), R61.2
- net q19_coll: now reaches J5.1 (Pin_1), Q19.2 (C), R60.1
- net rel_foot: now reaches D22.2 (A), J4.1 (Pin_1), K2.A2, R60.2
- net rel_mid: now reaches K1.A2, K2.A1
- new net +UB1_1: JP8.2 (B), K1.A1
Other:
- moved on the sheet: D22
